Commit message: robots works - PDDL to check

File: urdf/m2wr_arm2.xacro (robot description, xacro)
@@ -3,9 +3,9 @@
  <xacro:include filename="$(find erl2)/urdf/materials.xacro" />
  <xacro:include filename="$(find erl2)/urdf/m2wr_arm2.gazebo" />
- <xacro:macro name="cylinder_inertia" params="mass r l">
+<xacro:macro name="cylinder_inertia" params="mass r l">
     <inertia ixx="${mass*(3*r*r+l*l)/12}" ixy = "0" ixz = "0"
                 iyy="${mass*(3*r*r+l*l)/12}" iyz = "0" izz="${mass*(r*r)/2}" />
  </xacro:macro>
-   <xacro:macro name="link_wheel" params="name">
+    <xacro:macro name="link_wheel" params="name">
         <link name="${name}">
             <inertial>
